File: Hardware/AS5600 Breakout/AS5600 Breakout.sch (KiCad schematic (older format))
At the start: 6 parts, among them J1 Conn_01x08, U1 AS5600

Commit message: Completed breakout boards and BOM
Parts:
- removed J1: Conn_01x08, Pin_Headers:Pin_Header_Angled_1x08_Pitch2.54mm, symbol Conn_01x08
- added J1: Conn_01x07, Pin_Headers:Pin_Header_Angled_1x07_Pitch2.54mm, symbol Conn_01x07
Connections:
- net 5V: now also J1.7 (Pin_7)
- net DIR: now also J1.4 (Pin_4)
- net GND: now also J1.6 (Pin_6)
- net OUT: now also J1.5 (Pin_5)
- net PGO: now also J1.1 (Pin_1)
- net SCL: now also J1.3 (Pin_3)
- net SDA: now also J1.2 (Pin_2)
Changed lines of the file:
@@
-$EndComp
-$Comp
-L Conn_01x08 J1
-U 1 1 5B777435
-P 5450 2400
-F 0 "J1" H 5450 2800 50  0000 C CNN
-F 1 "Conn_01x08" V 5550 2400 50  0000 C CNN
-F 2 "Pin_Headers:Pin_Header_Angled_1x08_Pitch2.54mm" H 5450 2400 50  0001 C CNN
-F 3 "" H 5450 2400 50  0001 C CNN
-	1    5450 2400
-	0    -1   -1   0
 $EndComp
 $Comp
@@
 Wire Wire Line
 	6400 3300 6400 3350
+$Comp
+L Conn_01x07 J1
+U 1 1 5B78A669
+P 5450 2400
+F 0 "J1" V 5550 2750 50  0000 C CNN
+F 1 "Conn_01x07" V 5550 2250 50  0000 C CNN
+F 2 "Pin_Headers:Pin_Header_Angled_1x07_Pitch2.54mm" H 5450 2400 50  0001 C CNN
+F 3 "" H 5450 2400 50  0001 C CNN
+	1    5450 2400
+	0    1    -1   0
+$EndComp
 $EndSCHEMATC
